File: HB-UNI-Sen-TEMP-MAX6675.sch (KiCad schematic (older format))
At the start: 40 parts, among them IC1 CC1101, J1 TC1, J2 TC2, J3 FTDI, J4 Conn_01x02_Female, J5 AVR-ISP-6, SW1 Config, U1 MAX6675, U2 MAX6675, U3 ATmega328P-AU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

Commit message: Add files via upload
Parts:
- added JP6: VCC-Jumper, Jumper:SolderJumper-2_P1.3mm_Open_RoundedPad1.0x1.5mm, symbol Device:Jumper_NO_Small
- IC1: symbol homebrew:CC1101 -> HB-UNI-Sen-TEMP-MAX6675-rescue:CC1101-homebrew
- J5: symbol Connector:AVR-ISP-6 -> HB-UNI-Sen-TEMP-MAX6675-rescue:AVR-ISP-6-Connector
- JP5: value Jumper_NO_Small -> VCC-Jumper
- U1, U2: symbol homebrew:MAX6675 -> HB-UNI-Sen-TEMP-MAX6675-rescue:MAX6675-homebrew
- U3: symbol MCU_Microchip_ATmega:ATmega328P-AU -> HB-UNI-Sen-TEMP-MAX6675-rescue:ATmega328P-AU-MCU_Microchip_ATmega
- U4: symbol homebrew:MAX1724 -> HB-UNI-Sen-TEMP-MAX6675-rescue:MAX1724-homebrew
Connections:
- net VCC: now also JP6.1
- net at J3.3 (Pin_3): now also JP6.2
- no-connect marks 5 -> 4
Changed lines of the file:
@@
 EESchema Schematic File Version 4
+LIBS:HB-UNI-Sen-TEMP-MAX6675-cache
 EELAYER 30 0
 EELAYER END
@@
 $EndDescr
 $Comp
-L MCU_Microchip_ATmega:ATmega328P-AU U3
+L HB-UNI-Sen-TEMP-MAX6675-rescue:ATmega328P-AU-MCU_Microchip_ATmega U3
 U 1 1 5E2DF317
 P 7100 3400
@@
 $EndComp
 $Comp
-L homebrew:CC1101 IC1
+L HB-UNI-Sen-TEMP-MAX6675-rescue:CC1101-homebrew IC1
 U 1 1 5E2F7883
 P 10350 2000
@@
 $EndComp
 $Comp
-L homebrew:MAX1724 U4
+L HB-UNI-Sen-TEMP-MAX6675-rescue:MAX1724-homebrew U4
 U 1 1 5E2F8247
 P 3450 1800
@@
 MAX6675_SCK
 $Comp
-L homebrew:MAX6675 U2
+L HB-UNI-Sen-TEMP-MAX6675-rescue:MAX6675-homebrew U2
 U 1 1 5E2E1C21
 P 4450 4650
@@
 $EndComp
 $Comp
-L homebrew:MAX6675 U1
+L HB-UNI-Sen-TEMP-MAX6675-rescue:MAX6675-homebrew U1
 U 1 1 5E2E09ED
 P 1700 4650
@@
 	1500 1750 1250 1750
 $Comp
-L Connector:AVR-ISP-6 J5
+L HB-UNI-Sen-TEMP-MAX6675-rescue:AVR-ISP-6-Connector J5
 U 1 1 5E49F454
 P 1300 3450
@@
 Wire Wire Line
 	11050 2150 11050 2350
-NoConn ~ 7550 6150
 $Comp
 L Device:LED D1
@@
 P 1200 2750
 F 0 "JP5" V 1154 2798 50  0000 L CNN
-F 1 "Jumper_NO_Small" V 1245 2798 50  0000 L CNN
+F 1 "VCC-Jumper" V 1245 2798 50  0000 L CNN
 F 2 "Jumper:SolderJumper-2_P1.3mm_Open_RoundedPad1.0x1.5mm" H 1200 2750 50  0001 C CNN
 F 3 "~" H 1200 2750 50  0001 C CNN
@@
 Wire Wire Line
 	1200 2650 1200 2500
+$Comp
+L power:VCC #PWR0118
+U 1 1 5E4B8425
+P 7550 5425
+F 0 "#PWR0118" H 7550 5275 50  0001 C CNN
+F 1 "VCC" H 7650 5525 50  0000 C CNN
+F 2 "" H 7550 5425 50  0001 C CNN
+F 3 "" H 7550 5425 50  0001 C CNN
+	1    7550 5425
+	1    0    0    -1
+$EndComp
+$Comp
+L Device:Jumper_NO_Small JP6
+U 1 1 5E4B842C
+P 7550 5675
+F 0 "JP6" V 7504 5723 50  0000 L CNN
+F 1 "VCC-Jumper" V 7595 5723 50  0000 L CNN
+F 2 "Jumper:SolderJumper-2_P1.3mm_Open_RoundedPad1.0x1.5mm" H 7550 5675 50  0001 C CNN
+F 3 "~" H 7550 5675 50  0001 C CNN
+	1    7550 5675
+	0    1    1    0
+$EndComp
+Wire Wire Line
+	7550 5575 7550 5425
+Wire Wire Line
+	7550 5775 7550 6150
 $EndSCHEMATC

Commit message: Add files via upload
Other:
- note added: "CC BY-NC-SA 4.0"
Changed lines of the file:
@@
 Wire Wire Line
 	7550 5775 7550 6150
+Text Notes 8300 6925 0    118  ~ 24
+CC BY-NC-SA 4.0
 $EndSCHEMATC
