File: HB-UNI-Sen-TEMP-MAX6675.kicad_pcb (KiCad board)
At the start: 2 copper layers, 38.8 x 51.6 mm, 45 parts, among them IC1 CC1101, J1 TC1, J2 TC2, J3 FTDI, J4 Conn_01x02_Female, J5 AVR-ISP-6, SW1 Config, U1 MAX6675, U2 MAX6675, U3 ATmega328P-AU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

Commit message: Add files via upload
Parts:
- removed the REF** at (178.2, 70.8)
- removed the REF** at (144.2, 70.8)
- added JP6: VCC-Jumper, Jumper:SolderJumper-2_P1.3mm_Open_RoundedPad1.0x1.5mm, B.Cu at (148.7, 87.3)
- added REF**: MountingHole_2.1mm, MountingHole:MountingHole_2.1mm, F.Cu at (178.2, 72.9)
- added REF**: MountingHole_2.1mm, MountingHole:MountingHole_2.1mm, F.Cu at (144.2, 72.9)
- JP5: value Jumper_NO_Small -> VCC-Jumper
- moved J1 2.80 mm to (170.7, 74.6)
- moved J2 2.20 mm to (156.6, 74.6)
- moved JP2 1.99 mm to (170.7, 80.9)
- moved L2 1.99 mm to (170.7, 80.9)
- moved C7 1.99 mm to (168.2, 80.9)
- moved JP1 1.99 mm to (165.6, 80.9)
- moved L3 1.99 mm to (165.6, 80.9)
- moved D1 1.55 mm to (145.2, 98.3)
- moved J3 1.55 mm to (145.2, 80.0)
- moved J5 1.48 mm to (172.4, 112.3)
- moved C9 0.85 mm to (154.1, 80.9)
- moved JP3 0.85 mm to (156.6, 80.8)
- moved JP4 0.85 mm to (151.6, 80.9)
- moved L4 0.85 mm to (156.6, 80.8)
- moved L5 0.85 mm to (151.6, 80.9)
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Connections:
- JP1 pad 1: Net-(C7-Pad1) -> (no net)
- JP2 pad 1: Net-(C7-Pad2) -> (no net)
- JP3 pad 1: Net-(C9-Pad1) -> (no net)
- JP4 pad 1: Net-(C9-Pad2) -> (no net)
Routing:
- net VCC: track 104.0 -> 113.3 mm, vias 7 -> 6
- net /RESET: track 46.4 -> 52.8 mm, vias 3 -> 2
- net Net-(J3-Pad3): track 0.00 -> 4.64 mm
- net Net-(C10-Pad1): track 10.5 -> 7.72 mm
- net /TC_2-: track 8.04 -> 10.2 mm
- net /RX: track 19.8 -> 21.8 mm
- net /TC_1+: track 6.46 -> 8.44 mm
- net /SCLK: track 19.9 -> 18.3 mm
- net /MISO: track 16.9 -> 15.4 mm
- net Net-(C9-Pad1): track 9.12 -> 7.70 mm
- net Net-(C9-Pad2): track 10.1 -> 8.69 mm
- net /TC_2+: track 6.63 -> 8.04 mm
- net Net-(C7-Pad1): track 9.16 -> 7.75 mm
- net Net-(C7-Pad2): track 10.0 -> 8.62 mm
- net /TX: track 18.1 -> 16.8 mm
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- added copper zone on F.Cu, net GND
Other:
- board size 38.8 x 51.6 mm -> 38.8 x 49.6 mm
- board text added: "... der-pw/HB-UNI-Sen-TEMP-MAX6675-PCB"
- board text added: "... jp112sdl/HB-UNI-Sen-TEMP-MAX6675"
- board text added: "02/2020 der-pw CC BY-NC-SA 4.0"
- board text added: "FTDI"
- board text added: "cut Bridges"
- board text added: "https://github.com/..."
- board text added: "optional Filter"
- board text removed: "(c)2020 jp112sdl/der-pw CC BY-NC-SA 4.0"
- board text removed: "DTR"
- board text removed: "GND"
- board text removed: "NC"
- board text removed: "RX"
- board text removed: "TX"
- board text removed: "optional"

Commit message: Add files via upload
Changed lines of the file:
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@@
     (thickness 1.6)
     (drawings 36)
-    (tracks 405)
+    (tracks 404)
     (zones 0)
     (modules 46)
@@
     (add_net VCC)
   )
+  (module Connector_PinHeader_2.54mm:PinHeader_2x03_P2.54mm_Vertical (layer F.Cu)
+    (at 172.45 112.35 90)
+    (descr "Through hole straight pin header, 2x03, 2.54mm pitch, double rows")
+    (tags "Through hole pin header THT 2x03 2.54mm double row")
+    (fp_text reference J5 (at 1.27 -2.33 90) (layer F.SilkS) hide
+      (effects (font (size 1 1) (thickness 0.15)))
+    )
+    (fp_text value AVR-ISP-6 (at 1.27 7.41 90) (layer F.Fab)
+      (effects (font (size 1 1) (thickness 0.15)))
+    )
+    (fp_text user %R (at 1.27 2.54 180) (layer F.Fab)
+      (effects (font (size 1 1) (thickness 0.15)))
+    )
+    (fp_line (start 4.35 -1.8) (end -1.8 -1.8) (layer F.CrtYd) (width 0.05))
+    (fp_line (start 4.35 6.85) (end 4.35 -1.8) (layer F.CrtYd) (width 0.05))
+    (fp_line (start -1.8 6.85) (end 4.35 6.85) (layer F.CrtYd) (width 0.05))
+    (fp_line (start -1.8 -1.8) (end -1.8 6.85) (layer F.CrtYd) (width 0.05))
+    (fp_line (start 1.27 -1.33) (end 3.87 -1.33) (layer F.SilkS) (width 0.12))
+    (fp_line (start -1.33 1.27) (end -1.33 -1.33) (layer F.SilkS) (width 0.12))
+    (fp_line (start -1.33 -1.33) (end 1.27 -1.33) (layer F.SilkS) (width 0.12))
+    (fp_line (start 3.87 -1.33) (end 3.87 6.41) (layer F.SilkS) (width 0.12))
+    (fp_line (start -1.33 1.27) (end -1.33 6.41) (layer F.SilkS) (width 0.12))
+    (fp_line (start -1.33 6.41) (end 3.87 6.41) (layer F.SilkS) (width 0.12))
+    (fp_line (start -1.27 0) (end 0 -1.27) (layer F.Fab) (width 0.1))
+    (fp_line (start -1.27 6.35) (end -1.27 0) (layer F.Fab) (width 0.1))
+    (fp_line (start 3.81 6.35) (end -1.27 6.35) (layer F.Fab) (width 0.1))
+    (fp_line (start 3.81 -1.27) (end 3.81 6.35) (layer F.Fab) (width 0.1))
+    (fp_line (start 0 -1.27) (end 3.81 -1.27) (layer F.Fab) (width 0.1))
+    (fp_line (start 1.19 -1.32) (end 1.19 1.21) (layer F.SilkS) (width 0.15))
+    (fp_line (start -1.3 1.21) (end 1.19 1.21) (layer F.SilkS) (width 0.15))
+    (pad 6 thru_hole oval (at 2.4 5.08 90) (size 1.7 1.7) (drill 1) (layers *.Cu *.Mask)
+      (net 13 GND))
+    (pad 5 thru_hole oval (at -0.1 5.08 90) (size 1.7 1.7) (drill 1) (layers *.Cu *.Mask)
+      (net 33 /RESET))
+    (pad 4 thru_hole oval (at 2.6 2.54 90) (size 1.7 1.7) (drill 1) (layers *.Cu *.Mask)
+      (net 40 /MOSI))
+    (pad 3 thru_hole oval (at 0.1 2.54 90) (size 1.7 1.7) (drill 1) (layers *.Cu *.Mask)
+      (net 39 /SCLK))
+    (pad 2 thru_hole circle (at 2.4 0 90) (size 1.7 1.7) (drill 1) (layers *.Cu *.Mask)
+      (net 42 "Net-(J5-Pad2)"))
+    (pad 1 thru_hole rect (at -0.1 0 90) (size 1.7 1.7) (drill 1) (layers *.Cu *.Mask)
+      (net 38 /MISO))
+    (model ${KISYS3DMOD}/Connector_PinHeader_2.54mm.3dshapes/PinHeader_2x03_P2.54mm_Vertical.wrl
+      (at (xyz 0 0 0))
+      (scale (xyz 1 1 1))
+      (rotate (xyz 0 0 0))
+    )
+  )
   (module Jumper:SolderJumper-2_P1.3mm_Open_RoundedPad1.0x1.5mm (layer F.Cu)
     (at 169.25 108.25 270)
@@
       (net 13 GND))
     (model ${KISYS3DMOD}/Connector_PinHeader_2.54mm.3dshapes/PinHeader_1x02_P2.54mm_Vertical.wrl
-      (at (xyz 0 0 0))
-      (scale (xyz 1 1 1))
-      (rotate (xyz 0 0 0))
-    )
-  )
-  (module Connector_PinHeader_2.54mm:PinHeader_2x03_P2.54mm_Vertical (layer F.Cu)
-    (at 172.45 112.35 90)
-    (descr "Through hole straight pin header, 2x03, 2.54mm pitch, double rows")
-    (tags "Through hole pin header THT 2x03 2.54mm double row")
-    (fp_text reference J5 (at 1.27 -2.33 90) (layer F.SilkS) hide
-      (effects (font (size 1 1) (thickness 0.15)))
-    )
-    (fp_text value AVR-ISP-6 (at 1.27 7.41 90) (layer F.Fab)
-      (effects (font (size 1 1) (thickness 0.15)))
-    )
-    (fp_text user %R (at 1.27 2.54) (layer F.Fab)
-      (effects (font (size 1 1) (thickness 0.15)))
-    )
-    (fp_line (start 4.35 -1.8) (end -1.8 -1.8) (layer F.CrtYd) (width 0.05))
-    (fp_line (start 4.35 6.85) (end 4.35 -1.8) (layer F.CrtYd) (width 0.05))
-    (fp_line (start -1.8 6.85) (end 4.35 6.85) (layer F.CrtYd) (width 0.05))
-    (fp_line (start -1.8 -1.8) (end -1.8 6.85) (layer F.CrtYd) (width 0.05))
-    (fp_line (start 1.27 -1.33) (end 3.87 -1.33) (layer F.SilkS) (width 0.12))
-    (fp_line (start -1.33 1.27) (end -1.33 -1.33) (layer F.SilkS) (width 0.12))
-    (fp_line (start -1.33 -1.33) (end 1.27 -1.33) (layer F.SilkS) (width 0.12))
-    (fp_line (start 3.87 -1.33) (end 3.87 6.41) (layer F.SilkS) (width 0.12))
-    (fp_line (start -1.33 1.27) (end -1.33 6.41) (layer F.SilkS) (width 0.12))
-    (fp_line (start -1.33 6.41) (end 3.87 6.41) (layer F.SilkS) (width 0.12))
-    (fp_line (start -1.27 0) (end 0 -1.27) (layer F.Fab) (width 0.1))
-    (fp_line (start -1.27 6.35) (end -1.27 0) (layer F.Fab) (width 0.1))
-    (fp_line (start 3.81 6.35) (end -1.27 6.35) (layer F.Fab) (width 0.1))
-    (fp_line (start 3.81 -1.27) (end 3.81 6.35) (layer F.Fab) (width 0.1))
-    (fp_line (start 0 -1.27) (end 3.81 -1.27) (layer F.Fab) (width 0.1))
-    (pad 6 thru_hole oval (at 2.4 5.08 90) (size 1.7 1.7) (drill 1) (layers *.Cu *.Mask)
-      (net 13 GND))
-    (pad 5 thru_hole oval (at -0.1 5.08 90) (size 1.7 1.7) (drill 1) (layers *.Cu *.Mask)
-      (net 33 /RESET))
-    (pad 4 thru_hole oval (at 2.6 2.54 90) (size 1.7 1.7) (drill 1) (layers *.Cu *.Mask)
-      (net 40 /MOSI))
-    (pad 3 thru_hole oval (at 0.1 2.54 90) (size 1.7 1.7) (drill 1) (layers *.Cu *.Mask)
-      (net 39 /SCLK))
-    (pad 2 thru_hole rect (at 2.4 0 90) (size 1.7 1.7) (drill 1) (layers *.Cu *.Mask)
-      (net 42 "Net-(J5-Pad2)"))
-    (pad 1 thru_hole circle (at -0.1 0 90) (size 1.7 1.7) (drill 1) (layers *.Cu *.Mask)
-      (net 38 /MISO))
-    (model ${KISYS3DMOD}/Connector_PinHeader_2.54mm.3dshapes/PinHeader_2x03_P2.54mm_Vertical.wrl
       (at (xyz 0 0 0))
       (scale (xyz 1 1 1))
@@
   (segment (start 153.478552 83.803552) (end 151.647001 81.972001) (width 0.3) (layer F.Cu) (net 28))
   (segment (start 151.647001 81.972001) (end 151.56 81.972001) (width 0.3) (layer F.Cu) (net 28))
-  (segment (start 151.56 81.972001) (end 151.56 82.41) (width 0.3) (layer F.Cu) (net 28))
   (segment (start 177.3 98.725) (end 175.825 98.725) (width 0.25) (layer F.Cu) (net 29))
   (segment (start 175.05 97.95) (end 173.25 97.95) (width 0.25) (layer F.Cu) (net 29))

Commit message: update
forget a damn via
Routing:
- net VCC: vias 6 -> 7
Changed lines of the file:
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@@
     (thickness 1.6)
     (drawings 36)
-    (tracks 404)
+    (tracks 406)
     (zones 0)
     (modules 46)
@@
   (segment (start 157.586 89.3) (end 159.35 89.3) (width 0.25) (layer F.Cu) (net 11))
   (segment (start 169.25 104.5) (end 169.25 107.7) (width 0.3) (layer F.Cu) (net 11))
+  (segment (start 167.4 103.275) (end 167.4 103.275) (width 0.25) (layer F.Cu) (net 11))
+  (via (at 167.4 103.275) (size 0.8) (drill 0.4) (layers F.Cu B.Cu) (net 11))
   (segment (start 165.302 98.16) (end 164.252 98.16) (width 0.25) (layer F.Cu) (net 12))
   (segment (start 178.1 87.075) (end 175.6 87.075) (width 0.3) (layer F.Cu) (net 12))

Commit message: update
Other:
- net class Default removed
